File: unister.kicad_pcb (KiCad board)
At the start: 2 copper layers, 163.8 x 102.9 mm, 115 parts, among them J0 AC IN, J1 K1_DRY, J10 IN1_WET, J11 IN2_WET, J2 K1_230VAC, J3 K2_DRY, J4 K2_230VAC, J5 K3_DRY, J6 K3_230VAC, J7 K4_DRY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

Commit message: Revision 2: Grow fuses distance, move mounting holes
Parts:
- removed the ? at (66.0, 75.6)
- removed the ? at (63.5, 62.9)
- removed the ? at (63.5, 75.6)
- removed the ? at (66.0, 70.5)
- removed the ? at (66.0, 83.2)
- removed the ? at (66.0, 73.0)
- removed the ? at (63.5, 80.6)
- removed the ? at (66.0, 67.9)
- removed the ? at (66.0, 85.7)
- removed the ? at (63.5, 65.4)
- removed the ? at (63.5, 88.3)
- removed the ? at (63.5, 60.3)
- removed the ? at (63.5, 70.5)
- removed the ? at (66.0, 88.3)
- removed the ? at (66.0, 80.6)
- removed the ? at (66.0, 62.9)
- removed the ? at (63.5, 85.7)
- removed the ? at (63.5, 73.0)
- removed the ? at (63.5, 78.1)
- removed the ? at (63.5, 67.9)
- removed the ? at (66.0, 78.1)
- removed the ? at (63.5, 83.2)
- removed the ? at (66.0, 60.3)
- removed the ? at (66.0, 65.4)
- moved F1 9.19 mm to (174.5, 105.4), turned to 90 degrees
- moved C5 5.08 mm to (208.8, 122.6)
- moved D7 5.08 mm to (214.0, 121.6)
- moved D8 5.08 mm to (177.8, 117.5)
- moved R2 5.08 mm to (206.4, 111.1)
- moved R4 5.08 mm to (177.8, 111.1)
- moved U3 5.08 mm to (181.6, 103.5)
- moved C6 5.08 mm to (187.9, 122.6)
- moved D6 5.08 mm to (198.8, 117.5)
- moved D9 5.08 mm to (193.0, 121.6)
- moved R3 5.08 mm to (198.8, 111.1)
- moved R5 5.08 mm to (185.4, 111.1)
- moved U2 5.08 mm to (202.6, 103.5)
- moved F3 3.17 mm to (167.6, 124.9)
- moved H1 1.10 mm to (67.1, 54.0)
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Routing:
- net +5V: track 203.8 -> 210.6 mm
- net Net-(J0-Pin_3): track 56.6 -> 49.9 mm
- net Net-(TP17-Pad1): track 45.2 -> 49.9 mm
- net L_K34: track 80.8 -> 83.9 mm
- net GND: track 272.1 -> 269.0 mm
- net Earth_Protective: track 114.6 -> 117.4 mm
- net NEUT: track 205.6 -> 207.9 mm
- net Net-(D8-A): track 11.0 -> 8.89 mm
- net Net-(D6-A): track 11.0 -> 8.89 mm
- net Net-(D7-A): track 40.1 -> 41.6 mm
- net Net-(D9-A): track 40.1 -> 41.6 mm
- net Net-(PS1-AC/L): track 12.6 -> 13.7 mm

Commit message: Revision 2: Add print, export production files
Other:
- board text added: "Rev. 2"
Changed lines of the file:
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@@
 		(layer "Edge.Cuts")
+	)
+	(gr_text "Rev. 2"
+		(at 152.5 93.5 0)
+		(layer "F.SilkS")
+		(effects
+			(font
+				(size 2 2)
+				(thickness 0.15)
+			)
+			(justify left bottom)
+		)
 	)
 	(segment
